Commit message: simplification du robot reel

File: description/lidar.xacro (robot description, xacro)
@@ -1,8 +1,29 @@
 <?xml version="1.0"?>
 <robot xmlns:xacro="http://www.ros.org/wiki/xacro">
+    <joint name="support_joint" type="fixed">
+        <parent link="chassis"/>
+        <child link="support_frame"/>
+        <origin xyz="0.1 0 0.10545"/>
+    </joint>
+    <link name="support_frame">
+        <visual>
+            <geometry>
+                <box size="0.1 0.1 0.0839"/>
+            </geometry>
+            <material name="black"/>
+        </visual>
+        <collision>
+            <geometry>
+                <box size="0.1 0.1 0.0839"/>
+            </geometry>
+        </collision>
+        <xacro:inertial_box mass="0.1" x="0.1" y="0" z="0.175">
+            <origin xyz="0 0 0" rpy="0 0 0"/>
+        </xacro:inertial_box>
+    </link>
     <joint name="laser_joint" type="fixed">
-        <parent link="chassis"/>
+        <parent link="support_frame"/>
         <child link="laser_frame"/>
-        <origin xyz="0.1 0 0.175" rpy="0 0 0"/>
+        <origin xyz="0 0 0.06" rpy="0 0 0"/>
     </joint>
     <link name="laser_frame">
@@ -11,5 +32,5 @@
                 <cylinder radius="0.05" length="0.04" />
             </geometry>
-            <material name="orange"/>
+            <material name="blue"/>
         </visual>
         <collision>

File: description/robot.urdf.xacro (robot description, xacro)
@@ -3,4 +3,5 @@
     <xacro:include filename="robot_core.xacro" />
     <xacro:include filename="ros2_control.xacro"/>
+    <!--xacro:include filename="gazebo_control.xacro"/-->
     <xacro:include filename="lidar.xacro"/>
 </robot>

File: description/robot_core.xacro (robot description, xacro)
@@ -25,18 +25,18 @@
     <link name="chassis">
         <visual>
-            <origin xyz="0.15 0 0.075" rpy="0 0 0"/>
+            <origin xyz="0.15 0 0.03175" rpy="0 0 0"/>
             <geometry>
-                <box size="0.3 0.3 0.15"/>
+                <box size="0.38 0.365 0.0635"/>
             </geometry>
             <material name="white"/>
         </visual>
         <collision>
-            <origin xyz="0.15 0 0.075" rpy="0 0 0"/>
+            <origin xyz="0.15 0 0.03175" rpy="0 0 0"/>
             <geometry>
-                <box size="0.3 0.3 0.15"/>
+                <box size="0.38 0.365 0.0635"/>
             </geometry>
         </collision>
-        <xacro:inertial_box mass="0.5" x="0.3" y="0.3" z="0.15">
-            <origin xyz="0.15 0 0.75" rpy="0 0 0"/>
+        <xacro:inertial_box mass="0.5" x="0.38" y="0.365" z="0.0635">
+            <origin xyz="0.15 0 0.03175" rpy="0 0 0"/>
         </xacro:inertial_box>
     </link>
@@ -45,5 +45,5 @@
         <parent link="base_link"/>
         <child link="left_wheel"/>
-        <origin xyz="0 0.175 0" rpy="-${pi/2} 0 0"/>
+        <origin xyz="0 0.2025 -0.032" rpy="-${pi/2} 0 0"/>
         <axis xyz="0 0 1"/>
     </joint>
@@ -51,5 +51,5 @@
         <visual>
             <geometry>
-                <cylinder radius="0.05" length="0.04" />
+                <cylinder radius="0.018" length="0.04" />
             </geometry>
             <material name="orange"/>
@@ -57,8 +57,8 @@
         <collision>
             <geometry>
-                <cylinder radius="0.05" length="0.04" />
+                <cylinder radius="0.018" length="0.04" />
             </geometry>
         </collision>
-        <xacro:inertial_cylinder mass="0.1" length="0.04" radius="0.05">
+        <xacro:inertial_cylinder mass="0.1" length="0.04" radius="0.018">
             <origin xyz="0 0 0" rpy="0 0 0"/>
         </xacro:inertial_cylinder>
@@ -68,5 +68,5 @@
         <parent link="base_link"/>
         <child link="right_wheel"/>
-        <origin xyz="0 -0.175 0" rpy="${pi/2} 0 0"/>
+        <origin xyz="0 -0.2025 -0.032" rpy="${pi/2} 0 0"/>
         <axis xyz="0 0 -1"/>
     </joint>
@@ -74,5 +74,5 @@
         <visual>
             <geometry>
-                <cylinder radius="0.05" length="0.04" />
+                <cylinder radius="0.018" length="0.04" />
             </geometry>
             <material name="orange"/>
@@ -80,8 +80,8 @@
         <collision>
             <geometry>
-                <cylinder radius="0.05" length="0.04" />
+                <cylinder radius="0.018" length="0.04" />
             </geometry>
         </collision>
-        <xacro:inertial_cylinder mass="0.1" length="0.04" radius="0.05">
+        <xacro:inertial_cylinder mass="0.1" length="0.04" radius="0.018">
             <origin xyz="0 0 0" rpy="0 0 0"/>
         </xacro:inertial_cylinder>
@@ -91,5 +91,5 @@
         <parent link="chassis"/>
         <child link="caster_wheel"/>
-        <origin xyz="0.24 0 0"/>
+        <origin xyz="0.28 0 0"/>
     </joint>
     <link name="caster_wheel">
