Commit message: Reglage de la syncronisation entre gaz et rviz

File: description/gazebo_control.xacro (robot description, xacro)
@@ -5,9 +5,8 @@
             <left_joint> left_wheel_joint</left_joint>
             <right_joint> right_wheel_joint</right_joint>
-            <wheel_separation>0.35</wheel_separation>
-            <wheel_diameter>0.1</wheel_diameter>
+            <wheel_separation>0.405</wheel_separation>
+            <wheel_radius>0.018</wheel_radius> <!-- la dimention de la roue doit absolument etre en rayon et non en diametre!!! -->
             <!-- Limits -->
-            <max_wheel_torque>200</max_wheel_torque>
-            <max_wheel_acceleration>10.0</max_wheel_acceleration>
+            <max_wheel_acceleration>0.1</max_wheel_acceleration>
             <!-- Input -->
             <topic>cmd_vel</topic>

File: description/robot.urdf.xacro (robot description, xacro)
@@ -1,5 +1,5 @@
 <?xml version="1.0"?>
 <robot xmlns:xacro="http://www.ros.org/wiki/xacro"  name="robot">
-    <xacro:include filename="robot_core.xacro" />
+    <xacro:include filename="robot_core.xacro"/>
     <xacro:include filename="ros2_control.xacro"/>
     <!--xacro:include filename="gazebo_control.xacro"/-->

File: description/robot_core.xacro (robot description, xacro)
@@ -37,5 +37,5 @@
             </geometry>
         </collision>
-        <xacro:inertial_box mass="0.5" x="0.38" y="0.365" z="0.0635">
+        <xacro:inertial_box mass="5" x="0.38" y="0.365" z="0.0635">
             <origin xyz="0.15 0 0.03175" rpy="0 0 0"/>
         </xacro:inertial_box>
@@ -57,5 +57,5 @@
         <collision>
             <geometry>
-                <cylinder radius="0.018" length="0.04" />
+                <sphere radius="0.018"/>
             </geometry>
         </collision>
@@ -80,5 +80,5 @@
         <collision>
             <geometry>
-                <cylinder radius="0.018" length="0.04" />
+                <sphere radius="0.018"/>
             </geometry>
         </collision>
