Commit message: Gazebo

File: description/robot_core.xacro (robot description, xacro)
@@ -109,3 +109,8 @@
         </xacro:inertial_sphere>
     </link>
+    <gazebo reference="caster_wheel">
+        <material>Gazebo/Black</material>
+        <mu1 value="0.001"/>
+        <mu2 value="0.002"/>
+    </gazebo>
 </robot>

Commit message: Slam et Nav2

File: description/robot_core.xacro (robot description, xacro)
@@ -17,10 +17,18 @@
     <link name="base_link">
     </link>
+    <!-- Base foot print -->
+    <joint name="base_footprint_joint" type="fixed">
+        <parent link="base_link"/>
+        <child link="base_footprint"/>
+        <origin xyz="0 0 0" rpy="0 0 0"/>
+    </joint>
+    <link name="base_footprint">
+    </link>
+    <!-- Chassis link-->
     <joint name="chassis_joint" type="fixed">
-    <parent link="base_link"/>
-    <child link="chassis"/>
-    <origin xyz="-0.1 0 0"/>
+        <parent link="base_link"/>
+        <child link="chassis"/>
+        <origin xyz="-0.1 0 0"/>
     </joint>
-    <!-- Chassis link-->
     <link name="chassis">
         <visual>
